Commit message: fixd ES

File: assets/urdf/Armor_Robot/urdf/Armor_Robot.urdf (robot description, URDF)
Before this commit: robot Armor_Robot, 15 links, 14 joints
Links:
- added link Armor_num_link_1, mass 0.00034078; visual mesh filename=package://Armor_Robot/meshes/Armor_num_link_1.STL
- added link Armor_num_link_2, mass 0.000340775843454777; visual mesh filename=package://Armor_Robot/meshes/Armor_num_link_2.STL
- added link Armor_num_link_3, mass 0.00034077584345476; visual mesh filename=package://Armor_Robot/meshes/Armor_num_link_3.STL
- added link Armor_num_link_4, mass 0.00034078; visual mesh filename=package://Armor_Robot/meshes/Armor_num_link_4.STL
- link Armor_board_link_1: mass 0.0479070281599563 -> 0.048187
- link Armor_board_link_2: mass 0.0479070281599565 -> 0.0481867874495532
- link Armor_board_link_3: mass 0.0479070281599564 -> 0.0481867874495531
- link Armor_board_link_4: mass 0.0479070281599563 -> 0.048187
- link Armor_light_link_1: mass 0.00710803062860533 -> 0.007108
- link Armor_light_link_2: mass 0.00710803062860532 -> 0.007108
- link Armor_light_link_3: mass 0.00710803062860533 -> 0.007108
- link Armor_light_link_4: mass 0.00710803062860533 -> 0.007108
- link Armor_link_1: mass 0.0509456108266251 -> 0.050946
- link Armor_link_2: mass 0.0509456157055777 -> 0.050945615705612
- link Armor_link_3: mass 0.0509456108266248 -> 0.0509456108266588
- link Armor_link_4: mass 0.0509456157056193 -> 0.0509456157056531
Joints:
- added joint Armor_num_joint_1: type fixed, parent Armor_board_link_1, child Armor_num_link_1, origin xyz=0 0 0 rpy=0 0 0, axis 0 0 0
- added joint Armor_num_joint_2: type fixed, parent Armor_board_link_2, child Armor_num_link_2, origin xyz=0 0 0 rpy=0 0 0, axis 0 0 0
- added joint Armor_num_joint_3: type fixed, parent Armor_board_link_3, child Armor_num_link_3, origin xyz=0 0 0 rpy=0 0 0, axis 0 0 0
- added joint Armor_num_joint_4: type fixed, parent Armor_board_link_4, child Armor_num_link_4, origin xyz=0 0 0 rpy=0 0 0, axis 0 0 0
