Commit message: update gold ore

File: assets/urdf/Exchange_Station/urdf/Exchange_Station.urdf (robot description, URDF)
Before this commit: robot Exchange_Station, 15 links, 14 joints
Links:
- link base_link: geometry visual mesh filename=package://Exchange_Station/meshes/base_link.STL

File: assets/urdf/Gold/urdf/Gold.urdf (robot description, URDF)
Before this commit: robot Gold, 7 links, 6 joints
Links:
- link base_link: mass 7.642304 -> 0.5
